Commit message: bugfix for fixed joints

File: examples/03-spherical_joints/rpspsbot.urdf (robot description, URDF)
Before this commit: robot RPSPSBot, 6 links, 5 joints
Links:
- added link link5, mass 1
Joints:
- added joint j5: type fixed, parent link4, child link5, origin xyz=0.000000 0.000000 0.000000 rpy=-0.000000 0.000000 -0.000000
