Commit message: added grasp matrix example and improved examples

File: examples/02-update_model/rprbot.urdf (robot description, URDF)
Before this commit: robot RPBot, 3 links, 2 joints
Links:
- added link link2, mass 1
Joints:
- added joint j2: type revolute, parent link1, child link2, origin xyz=0.000000 0.000000 0.000000 rpy=-0.000000 0.000000 -0.000000, axis 1 0 0, limit lower=-2.967 upper=2.967 effort=176 velocity=1.7104
