Commit message: more tests

File: tests/urdf/rrpbot.urdf (robot description, URDF)
Before this commit: robot RRPBot, 4 links, 3 joints
Joints:
- joint j1: axis 0 1 0 -> 1 0 0; limit lower=-1.5707 upper=1.5707 effort=150 velocity=1.5709 -> lower=-2.5707 upper=2.5707 effort=250 velocity=1.5709; origin xyz=0.000000 0.000000 0.000000 rpy=-0.000000 0.000000 -0.000000 -> xyz=0.000000 0.000000 1.000000 rpy=-0.000000 0.000000 -0.000000

Commit message: added back IK functions and tested them

File: tests/urdf/rrpbot.urdf (robot description, URDF)
Before this commit: robot RRPBot, 4 links, 3 joints
Joints:
- joint j2: limit lower=0 upper=2.0 effort=200 velocity=1.0 -> lower=-0.9 upper=2.0 effort=200 velocity=1.0
