Commit message: renamed sai2 to sai

File: urdf_models/panda/panda_arm_allegro_left.urdf (robot description, URDF)
Before this commit: robot panda_arm_allegro, 29 links, 28 joints
Links:
- link index_0: geometry collision mesh filename=${SAI_MODEL_URDF_FOLDER}/allegro_hand/meshes/link_0.0.obj; visual mesh filename=${SAI_MODEL_URDF_FOLDER}/allegro_hand/meshes/link_0.0.obj
- link index_1: geometry collision mesh filename=${SAI_MODEL_URDF_FOLDER}/allegro_hand/meshes/link_1.0.obj; visual mesh filename=${SAI_MODEL_URDF_FOLDER}/allegro_hand/meshes/link_1.0.obj
- link index_2: geometry collision mesh filename=${SAI_MODEL_URDF_FOLDER}/allegro_hand/meshes/link_2.0.obj; visual mesh filename=${SAI_MODEL_URDF_FOLDER}/allegro_hand/meshes/link_2.0.obj
- link index_3: geometry collision mesh filename=${SAI_MODEL_URDF_FOLDER}/allegro_hand/meshes/link_3.0.obj; visual mesh filename=${SAI_MODEL_URDF_FOLDER}/allegro_hand/meshes/link_3.0.obj
- link index_tip: geometry collision sphere radius=0.012; visual mesh filename=${SAI_MODEL_URDF_FOLDER}/allegro_hand/meshes/link_3.0_tip.o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
- link middle_0: geometry collision mesh filename=${SAI_MODEL_URDF_FOLDER}/allegro_hand/meshes/link_0.0.obj; visual mesh filename=${SAI_MODEL_URDF_FOLDER}/allegro_hand/meshes/link_0.0.obj
- link middle_1: geometry collision mesh filename=${SAI_MODEL_URDF_FOLDER}/allegro_hand/meshes/link_1.0.obj; visual mesh filename=${SAI_MODEL_URDF_FOLDER}/allegro_hand/meshes/link_1.0.obj
- link middle_2: geometry collision mesh filename=${SAI_MODEL_URDF_FOLDER}/allegro_hand/meshes/link_2.0.obj; visual mesh filename=${SAI_MODEL_URDF_FOLDER}/allegro_hand/meshes/link_2.0.obj
- link middle_3: geometry collision mesh filename=${SAI_MODEL_URDF_FOLDER}/allegro_hand/meshes/link_3.0.obj; visual mesh filename=${SAI_MODEL_URDF_FOLDER}/allegro_hand/meshes/link_3.0.obj
- link middle_tip: geometry collision sphere radius=0.012; visual mesh filename=${SAI_MODEL_URDF_FOLDER}/allegro_hand/meshes/link_3.0_tip.o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
- link palm_link: geometry collision box size=0.0407 0.0785 0.093; visual mesh filename=${SAI_MODEL_URDF_FOLDER}/allegro_hand/meshes/base_link_left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
- link ring_0: geometry collision mesh filename=${SAI_MODEL_URDF_FOLDER}/allegro_hand/meshes/link_0.0.obj; visual mesh filename=${SAI_MODEL_URDF_FOLDER}/allegro_hand/meshes/link_0.0.obj
- link ring_1: geometry collision mesh filename=${SAI_MODEL_URDF_FOLDER}/allegro_hand/meshes/link_1.0.obj; visual mesh filename=${SAI_MODEL_URDF_FOLDER}/allegro_hand/meshes/link_1.0.obj
- link ring_2: geometry collision mesh filename=${SAI_MODEL_URDF_FOLDER}/allegro_hand/meshes/link_2.0.obj; visual mesh filename=${SAI_MODEL_URDF_FOLDER}/allegro_hand/meshes/link_2.0.obj
- link ring_3: geometry collision mesh filename=${SAI_MODEL_URDF_FOLDER}/allegro_hand/meshes/link_3.0.obj; visual mesh filename=${SAI_MODEL_URDF_FOLDER}/allegro_hand/meshes/link_3.0.obj
- link ring_tip: geometry collision sphere radius=0.012; visual mesh filename=${SAI_MODEL_URDF_FOLDER}/allegro_hand/meshes/link_3.0_tip.o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
- link thumb_0: geometry collision mesh filename=${SAI_MODEL_URDF_FOLDER}/allegro_hand/meshes/link_12.0_left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; visual mesh filename=${SAI_MODEL_URDF_FOLDER}/allegro_hand/meshes/link_12.0_left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
- link thumb_1: geometry collision mesh filename=${SAI_MODEL_URDF_FOLDER}/allegro_hand/meshes/link_13.0.obj; visual mesh filename=${SAI_MODEL_URDF_FOLDER}/allegro_hand/meshes/link_13.0.obj
- link thumb_2: geometry collision mesh filename=${SAI_MODEL_URDF_FOLDER}/allegro_hand/meshes/link_14.0.obj; visual mesh filename=${SAI_MODEL_URDF_FOLDER}/allegro_hand/meshes/link_14.0.obj
- link thumb_3: geometry collision mesh filename=${SAI_MODEL_URDF_FOLDER}/allegro_hand/meshes/link_15.0.obj; visual mesh filename=${SAI_MODEL_URDF_FOLDER}/allegro_hand/meshes/link_15.0.obj
- link thumb_tip: geometry collision sphere radius=0.012; visual mesh filename=${SAI_MODEL_URDF_FOLDER}/allegro_hand/meshes/link_15.0_tip.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

File: urdf_models/panda/panda_arm_allegro_right.urdf (robot description, URDF)
Before this commit: robot panda_arm_allegro, 29 links, 28 joints
Links:
- link index_0: geometry collision mesh filename=${SAI_MODEL_URDF_FOLDER}/allegro_hand/meshes/link_0.0.obj; visual mesh filename=${SAI_MODEL_URDF_FOLDER}/allegro_hand/meshes/link_0.0.obj
- link index_1: geometry collision mesh filename=${SAI_MODEL_URDF_FOLDER}/allegro_hand/meshes/link_1.0.obj; visual mesh filename=${SAI_MODEL_URDF_FOLDER}/allegro_hand/meshes/link_1.0.obj
- link index_2: geometry collision mesh filename=${SAI_MODEL_URDF_FOLDER}/allegro_hand/meshes/link_2.0.obj; visual mesh filename=${SAI_MODEL_URDF_FOLDER}/allegro_hand/meshes/link_2.0.obj
- link index_3: geometry collision mesh filename=${SAI_MODEL_URDF_FOLDER}/allegro_hand/meshes/link_3.0.obj; visual mesh filename=${SAI_MODEL_URDF_FOLDER}/allegro_hand/meshes/link_3.0.obj
- link index_tip: geometry collision sphere radius=0.012; visual mesh filename=${SAI_MODEL_URDF_FOLDER}/allegro_hand/meshes/link_3.0_tip.o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
- link middle_0: geometry collision mesh filename=${SAI_MODEL_URDF_FOLDER}/allegro_hand/meshes/link_0.0.obj; visual mesh filename=${SAI_MODEL_URDF_FOLDER}/allegro_hand/meshes/link_0.0.obj
- link middle_1: geometry collision mesh filename=${SAI_MODEL_URDF_FOLDER}/allegro_hand/meshes/link_1.0.obj; visual mesh filename=${SAI_MODEL_URDF_FOLDER}/allegro_hand/meshes/link_1.0.obj
- link middle_2: geometry collision mesh filename=${SAI_MODEL_URDF_FOLDER}/allegro_hand/meshes/link_2.0.obj; visual mesh filename=${SAI_MODEL_URDF_FOLDER}/allegro_hand/meshes/link_2.0.obj
- link middle_3: geometry collision mesh filename=${SAI_MODEL_URDF_FOLDER}/allegro_hand/meshes/link_3.0.obj; visual mesh filename=${SAI_MODEL_URDF_FOLDER}/allegro_hand/meshes/link_3.0.obj
- link middle_tip: geometry collision sphere radius=0.012; visual mesh filename=${SAI_MODEL_URDF_FOLDER}/allegro_hand/meshes/link_3.0_tip.o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
- link palm_link: geometry collision box size=0.0407 0.0785 0.093; visual mesh filename=${SAI_MODEL_URDF_FOLDER}/allegro_hand/meshes/base_link.obj
- link ring_0: geometry collision mesh filename=${SAI_MODEL_URDF_FOLDER}/allegro_hand/meshes/link_0.0.obj; visual mesh filename=${SAI_MODEL_URDF_FOLDER}/allegro_hand/meshes/link_0.0.obj
- link ring_1: geometry collision mesh filename=${SAI_MODEL_URDF_FOLDER}/allegro_hand/meshes/link_1.0.obj; visual mesh filename=${SAI_MODEL_URDF_FOLDER}/allegro_hand/meshes/link_1.0.obj
- link ring_2: geometry collision mesh filename=${SAI_MODEL_URDF_FOLDER}/allegro_hand/meshes/link_2.0.obj; visual mesh filename=${SAI_MODEL_URDF_FOLDER}/allegro_hand/meshes/link_2.0.obj
- link ring_3: geometry collision mesh filename=${SAI_MODEL_URDF_FOLDER}/allegro_hand/meshes/link_3.0.obj; visual mesh filename=${SAI_MODEL_URDF_FOLDER}/allegro_hand/meshes/link_3.0.obj
- link ring_tip: geometry collision sphere radius=0.012; visual mesh filename=${SAI_MODEL_URDF_FOLDER}/allegro_hand/meshes/link_3.0_tip.o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
- link thumb_0: geometry collision mesh filename=${SAI_MODEL_URDF_FOLDER}/allegro_hand/meshes/link_12.0_righ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; visual mesh filename=${SAI_MODEL_URDF_FOLDER}/allegro_hand/meshes/link_12.0_righ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
- link thumb_1: geometry collision mesh filename=${SAI_MODEL_URDF_FOLDER}/allegro_hand/meshes/link_13.0.obj; visual mesh filename=${SAI_MODEL_URDF_FOLDER}/allegro_hand/meshes/link_13.0.obj
- link thumb_2: geometry collision mesh filename=${SAI_MODEL_URDF_FOLDER}/allegro_hand/meshes/link_14.0.obj; visual mesh filename=${SAI_MODEL_URDF_FOLDER}/allegro_hand/meshes/link_14.0.obj
- link thumb_3: geometry collision mesh filename=${SAI_MODEL_URDF_FOLDER}/allegro_hand/meshes/link_15.0.obj; visual mesh filename=${SAI_MODEL_URDF_FOLDER}/allegro_hand/meshes/link_15.0.obj
- link thumb_tip: geometry collision sphere radius=0.012; visual mesh filename=${SAI_MODEL_URDF_FOLDER}/allegro_hand/meshes/link_15.0_tip.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
